File: PCB/aparte_pcb/midden/midden.kicad_sch (KiCad schematic)
At the start: 48 parts, among them J1 Conn_01x10_Socket, J10 Screw_Terminal_01x01, J11 Screw_Terminal_01x01, J2 Screw_Terminal_01x01, J3 Screw_Terminal_01x01, J4 Conn_01x10_Socket, J5 Conn_01x04_Socket, J6 Screw_Terminal_01x01, J7 Screw_Terminal_01x01, J8 Screw_Terminal_01x01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

Commit message: extra PCB changes
Multi-line description of commit,
feel free to be detailed.

Signed-off-by: Abel Tim <git@abeltim.com>
Changed lines of the file:
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@@
 (kicad_sch
-	(version 20231120)
+	(version 20250114)
 	(generator "eeschema")
-	(generator_version "8.0")
+	(generator_version "9.0")
 	(paper "A4")
+	(rectangle
+		(start 39.37 151.13)
+		(end 85.09 181.61)
+		(stroke
+			(width 0)
+			(type default)
+		)
+		(fill
+			(type none)
+		)
+	)
+	(text "MIDDEN\n"
+		(exclude_from_sim no)
+		(at 102.108 24.892 0)
+		(effects
+			(font
+				(size 2.54 2.54)
+			)
+		)
+	)
 	(junction
 		(at 38.1 128.27)
@@
 		)
 	)
-	(rectangle
-		(start 39.37 151.13)
-		(end 85.09 181.61)
-		(stroke
-			(width 0)
-			(type default)
-		)
-		(fill
-			(type none)
-		)
-	)
-	(text "MIDDEN\n"
-		(exclude_from_sim no)
-		(at 102.108 24.892 0)
-		(effects
-			(font
-				(size 2.54 2.54)
-			)
-		)
-	)
 	(global_label "pr3"
 		(shape input)
@@
 		)
 	)
+	(embedded_fonts no)
 )
