File: PCB/aparte_pcb/boven/boven.kicad_sch (KiCad schematic)
At the start: 51 parts, among them IC1 TSSP4038, IC10 TSSP4038, IC11 TSSP4038, IC12 TSSP4038, IC13 TSSP4038, IC14 TSSP4038, IC15 TSSP4038, IC16 TSSP4038, IC2 TSSP4038, IC3 TSSP4038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

Commit message: almost finished extra pcb
The pcb is designed to be single layerd for simplisity, but there are still two unconnected lines, GND and 5V are now both in two seperate sections. Can connect via an wire or update the PCB. Will not spend a lot of time on it now for it is not shure we will use an PCB or just a board with lots of wires on it.

Signed-off-by: Abel Tim <git@abeltim.com>
Changed lines of the file:
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@@
 (kicad_sch
-	(version 20231120)
+	(version 20250114)
 	(generator "eeschema")
-	(generator_version "8.0")
+	(generator_version "9.0")
 	(paper "A4")
+	(rectangle
+		(start 207.01 44.45)
+		(end 207.01 44.45)
+		(stroke
+			(width 0)
+			(type default)
+		)
+		(fill
+			(type none)
+		)
+	)
+	(text "BOVEN\n"
+		(exclude_from_sim no)
+		(at 155.702 21.336 0)
+		(effects
+			(font
+				(size 2.54 2.54)
+			)
+		)
+	)
 	(junction
 		(at 224.79 95.25)
@@
 		)
 	)
-	(rectangle
-		(start 207.01 44.45)
-		(end 207.01 44.45)
-		(stroke
-			(width 0)
-			(type default)
-		)
-		(fill
-			(type none)
-		)
-	)
-	(text "BOVEN\n"
-		(exclude_from_sim no)
-		(at 155.702 21.336 0)
-		(effects
-			(font
-				(size 2.54 2.54)
-			)
-		)
-	)
 	(global_label "gnd"
 		(shape input)
@@
 		)
 	)
+	(embedded_fonts no)
 )
