File: PCB/next-pcb/total/total.kicad_sch (KiCad schematic)
At the start: 217 parts, among them J1 progam, K1 TE_PCH-1xxx2M, U1 P8X32A-D40, U2 24LC256, U4 TCA9548APWR, U5 ATmega8-16P, U6 TCA9548APWR, Y1 P8X32A-D40, Y2 Crystal

Commit message: Changes to PCB
added some symboles did some changes.

Signed-off-by: Abel Tim <git@abeltim.com>
Parts:
- removed C10, C11, C23, C24, C25, C3, C5, C6, C9: 0.1uF, symbol Device:C
- removed C26, C27, C28, C29, C30, C31, C32, C33, C4, C7, C8: 1.0uF, symbol Device:C
- removed JP10, JP11, JP12, JP13, JP14, JP15, JP16, JP17, JP2, JP3, JP4, JP5, JP6, JP7, JP8, JP9: SolderJumper_3_Open, symbol Jumper:SolderJumper_3_Open
- removed R78, R79, R80, R81, R82, R83: 10K, symbol Device:R_US
- removed R84: PULL-UP, symbol Device:R_US
- added 3v3, 5v, 5v_1: ~, Lib:U1V10FX, symbol lib:U1V10FX
- added BT1: Battery, Connector_AMASS:AMASS_XT60-M_1x02_P7.20mm_Vertical, symbol Device:Battery
- added BT2: Battery, Connector_AMASS:AMASS_XT30UPB-F_1x02_P5.0mm_Vertical, symbol Device:Battery
- added C35, C36: 100nF, symbol Device:C_Polarized
- added C37, C38, C39, C40, C41, C43, C45, C47, C51, C52, C53, C54, C55, C56, C57, C58: 1uF, symbol Device:C_Polarized
- added C42, C44, C46, C48, C49, C50: 0.1uF, symbol Device:C
- added D33, D34: D, symbol Device:D
- added D36: GREEN_LED, symbol Device:LED
- added D37: RED_LED, symbol Device:LED
- added F1: Fuse, symbol Device:Fuse
- added JP1, JP10, JP11, JP12, JP13, JP14, JP15, JP16, JP17, JP2, JP3, JP4, JP5, JP6, JP7, JP8, JP9: SolderJumper_3_Bridged123, symbol Jumper:SolderJumper_3_Bridged123
- added K2: DIPxx-1Cxx-51x, Relay_THT:Relay_StandexMeder_DIP_LowProfile, symbol Relay:DIPxx-1Cxx-51x
- added R100, R101, R102, R103, R86, R87, R90, R91, R92, R93, R94, R95, R96, R97, R98, R99: 10K, symbol Device:R_US
- added R88, R89: 1K, symbol Device:R_US
- added SW2: SW_Push, symbol Switch:SW_Push
- added TH1: 10K, symbol Device:Thermistor_NTC
- added U7, U8: ATmega8-16P, Package_DIP:DIP-28_W7.62mm, symbol MCU_Microchip_ATmega:ATmega8-16P
- added U9: MAX17263xxTE, Package_DFN_QFN:DFN-14-1EP_3x3mm_P0.4mm_EP1.78x2.35mm, symbol Battery_Management:MAX17263xxTE
- added Y3, Y4: Crystal, symbol Device:Crystal
- added ds1, ds2, ds3, ds4, ds5, ds6, ds7, ds8: ~, Connector_PinHeader_2.54mm:PinHeader_1x04_P2.54mm_Vertical, symbol lib:HC-SR04
- C13, C14, C15, C16: value 1.0uF -> 0.1uF
- C2: value 1.0uF -> 0.47uF
- R23, R28, R29, R38, R39, R40: value 100K -> 100
- R41, R60, R61, R62, R63, R64, R65, R66, R67: value 100K -> 10K
- R54: value 100 -> 100K
- R55, R56, R57, R58, R59: value 100 -> 10K
- R72: value 10K -> PULL-UP
- R75: value 10K -> R_SENS
- R76, R77: value 10K -> ?ohm
Connections:
- net +12V: now also R76.1, 3v3.1 (VIN), 5v.1 (VIN), 5v_1.1 (VIN), D33.1 (K), K2.6, R88.1, R89.2
- net +3.3V: now also R23.1, R28.1, R29.1, R38.1, R39.1, R40.1, R64.1, R65.1, R66.1, R67.1, R68.1, R69.1, R70.1, R71.1, R72.2, JP1.2 (C), JP10.2 (C), JP11.2 (C), JP12.2 (C), JP13.2 (C), JP14.2 (C), JP15.2 (C), JP16.2 (C), JP2.2 (C), JP3.2 (C), JP4.2 (C), JP5.2 (C), JP6.2 (C), JP7.2 (C), JP8.2 (C), JP9.2 (C); no longer R54.1, R55.1, R56.1, R57.1, R58.1, R59.1, R76.1, R77.1, U6.21 (A2)
- net +5V: now also R10.2, R11.2, R12.2, R13.2, R14.2, R15.2, R16.2, R17.2, R2.2, R3.2, R4.2, R5.2, R6.2, R7.2, R8.2, R9.2, 5v.3 (VOUT), C35.1, C36.1, R86.1, R87.1, U7.20 (AVCC), U7.21 (AREF), U7.7 (VCC), U8.20 (AVCC), U8.21 (AREF), U8.7 (VCC), ds1.1 (VCC), ds2.1 (VCC), ds3.1 (VCC), ds4.1 (VCC), ds5.1 (VCC), ds6.1 (VCC), ds7.1 (VCC), ds8.1 (VCC)
- net GND: now also IR1.2 (GND), IR10.2 (GND), IR11.2 (GND), IR12.2 (GND), IR13.2 (GND), IR14.2 (GND), IR15.2 (GND), IR16.2 (GND), IR2.2 (GND), IR3.2 (GND), IR4.2 (GND), IR5.2 (GND), IR6.2 (GND), IR7.2 (GND), IR8.2 (GND), IR9.2 (GND), R75.2, U6.21 (A2), 3v3.2 (GND), 5v.2 (GND), C35.2, C36.2, C37.2, C38.2, C39.2, C40.2, C41.2, C42.2, C43.2, C44.2, C45.2, C46.2, C47.2, C48.2, C49.2, C50.2, C51.2, C52.2, C53.2, C54.2, C55.2, C56.2, C57.2, C58.2, U7.22 (AGND), U7.8 (GND), U8.22 (AGND), U8.8 (GND), ds1.4 (GND), ds2.4 (GND), ds3.4 (GND), ds4.4 (GND), ds5.4 (GND), ds6.4 (GND), ds7.4 (GND), ds8.4 (GND); no longer C1.2, C2.2
- net SCL: now also R74.2, U9.14 (SCL)
- net SDA: now also R73.2, U9.13 (SDA)
- net at CS9.6 (SCL), U6.20 (SC7): now also R56.2; no longer R68.2
- net at CS13.4 (SDA), U6.10 (SD3): now also R101.2; no longer R64.2
- net at CS13.5 (INT): now also R68.2
- net at CS13.6 (SCL), U6.11 (SC3): now also R60.2; no longer R72.2
- net at R31.1: now also JP5.1 (A)
- net at CS2.1 (VDD), R22.2: now also C44.1, C45.1
- net at CS4.1 (VDD), R27.2: now also C16.1, C41.1
- net at R62.1: now also JP15.1 (A)
- net at CS11.4 (SDA), U6.15 (SD5): now also R99.2; no longer R62.2
- net at CS1.1 (VDD), R18.2: now also C46.1, C47.1; no longer C1.1, C2.1
- net at CS10.4 (SDA), U6.17 (SD6): now also R98.2; no longer R61.2
- net at CS10.5 (INT): now also R65.2; no longer R77.2
- net at CS10.6 (SCL), U6.18 (SC6): now also R57.2; no longer R69.2
- net at CS7.1 (VDD), R36.2: now also C13.1, C38.1; no longer C15.1
- net at CS7.4 (SDA), U4.6 (SD1): now also R90.2; no longer R40.2
- net at CS6.4 (SDA), U4.8 (SD2): now also R91.2; no longer R39.2
- net at R30.1: now also JP6.1 (A)
- net at CS3.1 (VDD), R26.2: now also C42.1, C43.1
- net at CS16.1 (VDD): now also C22.1, R53.2, C58.1; no longer R59.2
- net at CS16.4 (SDA), U6.4 (SD0): now also R55.2; no longer R67.2
- net at R44.1: now also JP2.1 (A)
- net at CS15.5 (INT): now also R70.2
- net at R58.2: now also CS11.6 (SCL), U6.16 (SC5); no longer CS15.1 (VDD)
- net at CS15.4 (SDA), U6.6 (SD1): now also R103.2; no longer R66.2
- net at CS15.6 (SCL), U6.7 (SC1): now also R62.2; no longer R74.2
- net at CS5.4 (SDA), U4.10 (SD3): now also R92.2; no longer R38.2
- net at CS4.4 (SDA), U4.13 (SD4): now also R93.2; no longer R29.2
- net at CS3.4 (SDA), U4.15 (SD5): now also R94.2; no longer R28.2
- net at CS2.4 (SDA), U4.17 (SD6): now also R95.2; no longer R23.2
- net at CS1.4 (SDA), R19.2, U4.19 (SD7): now also R96.2
- net at C14.1, CS6.1 (VDD), R35.2: now also C39.1
- net at CS11.5 (INT): now also R66.2
- net GND1: now reaches R75.1
- net GND1: now also C1.2, R77.2, 5v_1.2 (GND), D36.1 (K), K2.14, K2.2, SW2.1, TH1.2, U9.15 (EP), U9.8 (GND)
- net at CS16.6 (SCL), U6.5 (SC0): now also R63.2; no longer R75.2
- net at C12.1, CS8.1 (VDD), R37.2: now also C37.1; no longer C16.1
- net at CS12.4 (SDA), U6.13 (SD4): now also R100.2; no longer R63.2
- net at CS12.6 (SCL), U6.14 (SC4): now also R59.2; no longer R71.2
- net at CS9.4 (SDA), U6.19 (SD7): now also R54.2, R97.2; no longer R60.2
- net at U6.3 (~{RESET}): now also R72.1
- net at CS14.4 (SDA), U6.8 (SD2): now also R102.2; no longer R65.2
- net at CS14.6 (SCL), U6.9 (SC2): now also R61.2; no longer R73.2
- net at R73.1: now also JP17.1 (A)
- net at CS14.5 (INT): now also R69.2
- net at CS14.1 (VDD): now also C20.1, R40.2, C56.1; no longer R57.2
- net at CS12.5 (INT): now also R67.2
- net at R24.1: now also JP7.1 (A)
- net at R61.1: now also JP14.1 (A)
- net at R74.1: now also JP17.3 (B)
- net at R76.2: now also R77.1, U9.10 (CELLX/CSPH); no longer CS9.5 (INT)
- net at R43.1: now also JP3.1 (A)
- net at R60.1: now also JP13.1 (A)
- net at R63.1: now also JP16.1 (A)
- net at R45.1: now also JP1.1 (A)
- net at R41.1: now also JP1.3 (B)
- net at CS5.1 (VDD), R34.2: now also C15.1, C40.1; no longer C13.1
- net at CS16.5 (INT): now also R71.2
- net at R19.1: now also JP8.3 (B), R96.1
- net at R42.1: now also JP4.1 (A)
- net at R20.1: now also JP8.1 (A)
- net IR1: no longer names the net of IR1.1 (OUT)
- net IR1: now also U7.14 (PB0)
- net IR10: no longer names the net of IR10.1 (OUT)
- net IR10: now also U7.26 (PC3)
- net IR11: no longer names the net of IR11.1 (OUT)
- net IR11: now also U7.27 (PC4)
- net IR12: no longer names the net of IR12.1 (OUT)
- net IR12: now also U7.28 (PC5)
- net IR13: no longer names the net of IR13.1 (OUT)
- net IR13: now also U7.4 (PD2)
- net IR14: no longer names the net of IR14.1 (OUT)
- net IR14: now also U7.5 (PD3)
- net IR15: no longer names the net of IR15.1 (OUT)
- net IR15: now also U7.6 (PD4)
- net IR16: no longer names the net of IR16.1 (OUT)
- net IR16: now also U7.11 (PD5)
- net IR2: no longer names the net of IR2.1 (OUT)
- net IR2: now also U7.15 (PB1)
- net IR3: no longer names the net of IR3.1 (OUT)
- net IR3: now also U7.16 (PB2)
- net IR4: no longer names the net of IR4.1 (OUT)
- net IR4: now also U7.17 (PB3)
- net IR5: no longer names the net of IR5.1 (OUT)
- net IR5: now also U7.18 (PB4)
- net IR6: no longer names the net of IR6.1 (OUT)
- net IR6: now also U7.19 (PB5)
- net IR7: no longer names the net of IR7.1 (OUT)
- net IR7: now also U7.23 (PC0)
- net IR8: no longer names the net of IR8.1 (OUT)
- net IR8: now also U7.24 (PC1)
- net IR9: no longer names the net of IR9.1 (OUT)
- net IR9: now also U7.25 (PC2)
- new net: C50.1, C53.1, CS11.1 (VDD), R29.2
- new net: C19.1, C55.1, CS13.1 (VDD), R39.2
- new net: C48.1, C51.1, CS9.1 (VDD), R23.2
- new net: JP3.3 (B), R91.1
- new net: BT1.1 (+), BT2.1 (+), D33.2 (A)
- new net: BT1.2 (-), BT2.2 (-), D34.1 (K)
- new net: U8.25 (PC2), ds5.2 (Trig)
- new net: U8.26 (PC3), ds5.3 (Echo)
- new net: JP4.3 (B), R92.1
- new net: JP5.3 (B), R93.1
- new net: C49.1, C52.1, CS10.1 (VDD), R28.2
- new net: JP11.1 (A), R58.1
- new net: C18.1, C54.1, CS12.1 (VDD), R38.2
- new net: JP13.3 (B), R101.1
- new net: C2.2, U9.11 (REG)
- new net: JP14.3 (B), R102.1
- new net: U7.10 (PB7/XTAL2), Y3.1
- new net: U7.9 (PB6/XTAL1), Y3.2
- new net: U8.4 (PD2), ds7.2 (Trig)
- new net: U8.5 (PD3), ds7.3 (Echo)
- new net: R87.2, U8.1 (PC6/~{RESET})
- new net: U8.10 (PB7/XTAL2), Y4.1
- new net: U8.11 (PD5), ds8.3 (Echo)
- new net: U8.14 (PB0), ds1.2 (Trig)
- new net: U8.15 (PB1), ds1.3 (Echo)
- new net: U8.16 (PB2), ds2.2 (Trig)
- new net: U8.17 (PB3), ds2.3 (Echo)
- new net: U8.18 (PB4), ds3.2 (Trig)
- new net: U8.19 (PB5), ds3.3 (Echo)
- new net: U8.23 (PC0), ds4.2 (Trig)
- new net: U8.24 (PC1), ds4.3 (Echo)
- new net: U8.27 (PC4), ds6.2 (Trig)
- new net: U8.28 (PC5), ds6.3 (Echo)
- new net: U8.6 (PD4), ds8.2 (Trig)
- new net: U8.9 (PB6/XTAL1), Y4.2
- new net: TH1.1, U9.1 (TH)
- new net: 5v_1.3 (VOUT), C1.1, U9.6 (BATT)
- new net: JP9.3 (B), R54.1, R97.1
- new net: D37.1 (K), K2.1
- new net: D37.2 (A), R88.2
- new net: JP7.3 (B), R95.1
- new net: C21.1, C57.1, CS15.1 (VDD), R52.2
- new net: R86.2, U7.1 (PC6/~{RESET})
- new net: JP9.1 (A), R56.1
- new net: JP16.3 (B), R55.1
- new net: D36.2 (A), R89.1
- new net: JP15.3 (B), R103.1
- new net: JP10.3 (B), R98.1
- new net: JP6.3 (B), R94.1
- new net: D34.2 (A), F1.1
- new net: F1.2, K2.7, K2.8, SW2.2
- new net: JP12.1 (A), R59.1
- new net: JP12.3 (B), R100.1
- new net: JP11.3 (B), R99.1
- new net: JP2.3 (B), R90.1
- new net: JP10.1 (A), R57.1
- new net: CS9.5 (INT), R64.2
- new net +3V3: 3v3.3 (VOUT), JP17.2 (C)
- new net BATT_ALRT: U9.12 (ALRT)
- new net RX_DS: U8.2 (PD0)
- new net RX_IR: U7.2 (PD0)
- new net TX_DS: U8.3 (PD1)
- new net TX_IR: U7.3 (PD1)
Other:
- note added: "https://mm.digikey.com/Volume0/opasdata/d220001/medias/docus/7030/175_MAX17261.PDF"
- note added: "https://www.renesas.com/en/document/dst/isl29125-datasheet"
- note added: "https://www.scribd.com/document/698487550/short-circuit-protection-using-relay"
- moved on the sheet: C12, C17, C34, CS1, CS2, CS3, CS4, CS5, CS6, CS7, CS8, D1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
