File: PCB/aparte_pcb/extra_board/extra_board.kicad_pcb (KiCad board)
At the start: 2 copper layers, 9 parts, among them J1 Conn_01x10_Pin, J2 Conn_01x04_Pin, J3 Conn_01x10_Pin, J4 Conn_01x04_Pin, U2 MCP23017_SP

Commit message: recenltly removed three commit becouse it included files that shouldn't be included.
Did reset hard,
localy unstaged commits, deleted files and recommited the good files.
think this is all i did since,
-changed extra PCB name to bave and _ instead of a space so i dont have to use ""
-added button and led to teensy41 goaly overlay
-started on PWM, not complete

Abel Tim <git@abeltim.com>
Parts:
- added U3: PCA9685PW, Package_SO:TSSOP-28_4.4x9.7mm_P0.65mm, F.Cu at (3.88, 5.12)
- U1: value ~ -> soccer communinication module
Connections:
- net pr1 renamed /pr1
- net pr2 renamed /pr2
- net pr3 renamed /pr3
- net pr4 renamed /pr4
- net pr5 renamed /pr5
- net pr6 renamed /pr6
- net pr7 renamed /pr7
- net pr8 renamed /pr8
- DR2 pad 1: 12V -> +12V
- J1 pad 1: SCL -> GND
- J1 pad 10: GND -> /SCL
- J1 pad 2: RX -> /D-A1
- J1 pad 3: TX -> /D+A0
- J1 pad 4: encA -> /OUT1
- J1 pad 5: encB -> /OUT2
- J1 pad 6: OUT2 -> /encA
- J1 pad 7: D+A0 -> /encB
- J1 pad 8: D-A1 -> /TX
- J1 pad 9: GND -> /RX
- J2 pad 1: SDA -> /SDA
- J2 pad 3: 5v -> +5V
- J3 pad 1: Groen -> /GREEN
- J3 pad 2: Rood -> /RED
- J4 pad 1: blauw -> /BLUE
- J4 pad 3: 5v -> +5V
- M2 pad 4: 5v -> +5V
- M2 pad 5: encA -> /encA
- M2 pad 6: encB -> /encB
- U1 pad 1: unconnected-(U1-BAt+-Pad1) -> +12V
- U1 pad 10: OUT1 -> /OUT1
- U1 pad 2: 5v -> +5V
- U1 pad 5: D-A1 -> /D-A1
- U1 pad 6: D+A0 -> /D+A0
- U1 pad 9: OUT2 -> /OUT2
- adc1 pad 14: 5v -> unconnected-(adc1-5V-Pad14)
- adc1 pad 7: RX -> /RX
- adc1 pad 8: TX -> /TX
Routing:
- net (no net): track 0.00 -> 566.3 mm
- net TX: track 173.7 -> 0.00 mm
- net RX: track 153.5 -> 0.00 mm
- net encA: track 128.0 -> 0.00 mm
- net encB: track 111.1 -> 0.00 mm
